File: STM32G031J6M6/stm32G031J6M6-Breakout.sch (EAGLE design)
At the start: 25 parts, among them IC1 LDL112D33R, J2 PWR

Commit message: switched packages for caps so I could only work with 1/64 inch bits
Parts:
- C1, C2, C3, C4: device passives:C-USC0805 -> passives:C-USC0805K
Changed lines of the file:
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@@
 <parts>
 <part name="U$1" library="ICs" deviceset="STM32G031" device="S08N" package3d_urn="urn:adsk.eagle:package:16126582/1"/>
-<part name="C1" library="passives" deviceset="C-US" device="C0805" package3d_urn="urn:adsk.eagle:package:8118586/1" value="4.7 uF"/>
-<part name="C2" library="passives" deviceset="C-US" device="C0805" package3d_urn="urn:adsk.eagle:package:8118586/1" value="0.1 uF"/>
+<part name="C1" library="passives" deviceset="C-US" device="C0805K" package3d_urn="urn:adsk.eagle:package:8089589/1" value="4.7 uF"/>
+<part name="C2" library="passives" deviceset="C-US" device="C0805K" package3d_urn="urn:adsk.eagle:package:8089589/1" value="0.1 uF"/>
 <part name="IC1" library="voltage-regulator" deviceset="LDL112D33R" device=""/>
 <part name="S1" library="switches" deviceset="MSS3-V-T_R" device=""/>
-<part name="C3" library="passives" deviceset="C-US" device="C0805" package3d_urn="urn:adsk.eagle:package:8118586/1" value="10 uF"/>
+<part name="C3" library="passives" deviceset="C-US" device="C0805K" package3d_urn="urn:adsk.eagle:package:8089589/1" value="10 uF"/>
 <part name="J1" library="connector" deviceset="M08X2" device=""/>
 <part name="R1" library="passives" deviceset="RESISTOR" device="1206" value="56 R"/>
@@
 <part name="R9" library="passives" deviceset="RESISTOR" device="1206" value="56 R"/>
 <part name="U$2" library="switches" deviceset="SWITCH_TACTILE" device="TACTILE-2PIN-NARROW"/>
-<part name="C4" library="passives" deviceset="C-US" device="C0805" package3d_urn="urn:adsk.eagle:package:8118586/1" value="0.1 uF"/>
+<part name="C4" library="passives" deviceset="C-US" device="C0805K" package3d_urn="urn:adsk.eagle:package:8089589/1" value="0.1 uF"/>
 <part name="LED1" library="leds" deviceset="LED" device="1206"/>
 <part name="LED2" library="leds" deviceset="LED" device="1206"/>

Commit message: removed reset button as it was wrong AND don't need it
Parts:
- removed C4: 0.1 uF, passives:C-USC0805K
- removed R3: 10 K, passives:RESISTOR0805-RES
- removed U$2: SWITCH_TACTILETACTILE-2PIN-NARROW, switches:SWITCH_TACTILETACTILE-2PIN-NARROW
Connections:
- removed net N$1: C4.1, R3.1, U$2.A
- net GND: no longer C4.2, U$2.C
- net VDD: no longer R3.2

Commit message: adding rgb breakout
Connections:
- removed net N$16: IC1.EN, LED7.C
- net GND: now also LED7.C
- net N$14: now also IC1.EN
Other:
- moved on the sheet: LED7, R1
Changed lines of the file:
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@@
 <attribute name="NAME" x="48.26" y="29.21" size="1.778" layer="95"/>
 </instance>
-<instance part="R1" gate="G$1" x="134.62" y="35.56" smashed="yes">
-<attribute name="NAME" x="130.81" y="37.0586" size="1.778" layer="95"/>
-<attribute name="VALUE" x="130.81" y="32.258" size="1.778" layer="96"/>
+<instance part="R1" gate="G$1" x="144.78" y="35.56" smashed="yes">
+<attribute name="NAME" x="140.97" y="37.0586" size="1.778" layer="95"/>
+<attribute name="VALUE" x="140.97" y="32.258" size="1.778" layer="96"/>
 </instance>
 <instance part="R2" gate="G$1" x="5.08" y="25.4" smashed="yes">
@@
 <attribute name="VALUE" x="-29.972" y="6.985" size="1.778" layer="96"/>
 </instance>
-<instance part="LED7" gate="G$1" x="144.78" y="35.56" smashed="yes" rot="R90">
-<attribute name="NAME" x="149.352" y="39.116" size="1.778" layer="95" rot="R180"/>
-<attribute name="VALUE" x="149.352" y="41.275" size="1.778" layer="96" rot="R180"/>
+<instance part="LED7" gate="G$1" x="154.94" y="35.56" smashed="yes" rot="R90">
+<attribute name="NAME" x="159.512" y="39.116" size="1.778" layer="95" rot="R180"/>
+<attribute name="VALUE" x="159.512" y="41.275" size="1.778" layer="96" rot="R180"/>
 </instance>
 <instance part="J2" gate="G$1" x="172.72" y="30.48" smashed="yes" rot="R270">
@@
 <label x="177.8" y="20.32" size="1.778" layer="95"/>
 </segment>
+<segment>
+<pinref part="LED7" gate="G$1" pin="C"/>
+<wire x1="160.02" y1="35.56" x2="160.02" y2="33.02" width="0.1524" layer="91"/>
+<label x="160.02" y="30.48" size="1.778" layer="95"/>
+</segment>
 </net>
 <net name="VIN" class="0">
@@
 <segment>
 <pinref part="R1" gate="G$1" pin="1"/>
-<wire x1="129.54" y1="35.56" x2="124.46" y2="35.56" width="0.1524" layer="91"/>
-<label x="124.46" y="35.56" size="1.778" layer="95"/>
+<wire x1="139.7" y1="35.56" x2="137.16" y2="35.56" width="0.1524" layer="91"/>
+<label x="134.62" y="35.56" size="1.778" layer="95"/>
 </segment>
 </net>
@@
 <pinref part="R1" gate="G$1" pin="2"/>
 <pinref part="LED7" gate="G$1" pin="A"/>
-<wire x1="142.24" y1="35.56" x2="139.7" y2="35.56" width="0.1524" layer="91"/>
-</segment>
-</net>
-<net name="N$16" class="0">
-<segment>
-<pinref part="LED7" gate="G$1" pin="C"/>
+<wire x1="152.4" y1="35.56" x2="149.86" y2="35.56" width="0.1524" layer="91"/>
 <pinref part="IC1" gate="G$1" pin="EN"/>
 <wire x1="149.86" y1="35.56" x2="149.86" y2="45.72" width="0.1524" layer="91"/>
-</segment>
-</net>
+<junction x="149.86" y="35.56"/>
+</segment>
+</net>
